Commit message: Add experimental GRiD backend support

File: mpx/data/aliengo/aliengo.urdf (robot description, URDF)
Before this commit: robot aliengo, 31 links, 30 joints
Links:
- removed link base
- removed link imu_link
- link FL_calf: geometry collision box size=0.25 0.0208 0.016; visual mesh filename=assets/calf.stl scale=1 1 1
- link FL_hip: geometry collision cylinder length=0.0418 radius=0.046; visual mesh filename=assets/hip.stl scale=1 1 1
- link FL_thigh: geometry collision box size=0.25 0.0374 0.043; visual mesh filename=assets/thigh.stl scale=1 1 1
- link FR_calf: geometry collision box size=0.25 0.0208 0.016; visual mesh filename=assets/calf.stl scale=1 1 1
- link FR_hip: geometry collision cylinder length=0.0418 radius=0.046; visual mesh filename=assets/hip.stl scale=1 1 1
- link FR_thigh: geometry collision box size=0.25 0.0374 0.043; visual mesh filename=assets/thigh_mirror.stl scale=1 1 1
- link RL_calf: geometry collision box size=0.25 0.0208 0.016; visual mesh filename=/home/iit.local/abratta/dls1_noetic/src/quadruped_pympc_ros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 scale=1 1 1
- link RL_hip: geometry collision cylinder length=0.0418 radius=0.046; visual mesh filename=/home/iit.local/abratta/dls1_noetic/src/quadruped_pympc_ros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 scale=1 1 1
- link RL_thigh: geometry collision box size=0.25 0.0374 0.043; visual mesh filename=/home/iit.local/abratta/dls1_noetic/src/quadruped_pympc_ros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 scale=1 1 1
- link RR_calf: geometry collision box size=0.25 0.0208 0.016; visual mesh filename=assets/calf.stl scale=1 1 1
- link RR_hip: geometry collision cylinder length=0.0418 radius=0.046; visual mesh filename=assets/hip.stl scale=1 1 1
- link RR_thigh: geometry collision box size=0.25 0.0374 0.043; visual mesh filename=assets/thigh_mirror.stl scale=1 1 1
- link trunk: geometry collision box size=0.647 0.15 0.112; visual mesh filename=assets/trunk.stl scale=1 1 1
Joints:
- removed joint floating_base
- removed joint imu_joint
- joint FL_thigh_joint: limit effort=35.278 velocity=20 -> lower=-3.14 upper=3.14 effort=35.278 velocity=20; type continuous -> revolute
- joint FR_thigh_joint: limit effort=35.278 velocity=20 -> lower=-3.14 upper=3.14 effort=35.278 velocity=20; type continuous -> revolute
- joint RL_thigh_joint: limit effort=35.278 velocity=20 -> lower=-3.14 upper=3.14 effort=35.278 velocity=20; type continuous -> revolute
- joint RR_thigh_joint: limit effort=35.278 velocity=20 -> lower=-3.14 upper=3.14 effort=35.278 velocity=20; type continuous -> revolute
